Commit message: completed A.002 and A.003 diff_params.yaml modifies wheel radius and separation

File: nuturtle_description/urdf/turtlebot3_burger.gazebo.xacro (robot description, xacro)
@@ -3,4 +3,12 @@
   <xacro:arg name="laser_visual" default="false"/>
   <xacro:arg name="imu_visual"   default="false"/>
+  <!-- Load from yaml file -->
+  <xacro:property name='myyaml' value='$(find nuturtle_description)/config/diff_params.yaml'/>
+  <xacro:property name='diff_params' value='${load_yaml(myyaml)}'/>
+  <!-- wheel radius and separation -->
+  <!-- default WR=0.033 -->
+  <xacro:property name='WR' value='${diff_params["wheel_radius"]}'/>
+  <!-- default WS=0.16 -->
+  <xacro:property name='WS' value='${diff_params["wheel_base"]}'/>
   <gazebo reference="base_link">
     <material>Gazebo/DarkGrey</material>
@@ -57,6 +65,6 @@
       <leftJoint>wheel_left_joint</leftJoint>
       <rightJoint>wheel_right_joint</rightJoint>
-      <wheelSeparation>0.160</wheelSeparation>
-      <wheelDiameter>0.066</wheelDiameter>
+      <wheelSeparation>${WS}</wheelSeparation>
+      <wheelDiameter>${2*WR}</wheelDiameter>
       <wheelAcceleration>1</wheelAcceleration>
       <wheelTorque>10</wheelTorque>

File: nuturtle_description/urdf/turtlebot3_burger.urdf.xacro (robot description, xacro)
@@ -3,4 +3,12 @@
   <xacro:include filename="$(find nuturtle_description)/urdf/common_properties.xacro"/>
   <xacro:include filename="$(find nuturtle_description)/urdf/turtlebot3_burger.gazebo.xacro"/>
+  <!-- Load from yaml file -->
+  <xacro:property name='myyaml' value='$(find nuturtle_description)/config/diff_params.yaml'/>
+  <xacro:property name='diff_params' value='${load_yaml(myyaml)}'/>
+  <!-- wheel radius and separation -->
+  <!-- default WR=0.033 -->
+  <xacro:property name='WR' value='${diff_params["wheel_radius"]}'/>
+  <!-- default WS=0.16 -->
+  <xacro:property name='WS' value='${diff_params["wheel_base"]}'/>
   <link name="base_footprint"/>
   <joint name="base_joint" type="fixed">
@@ -34,5 +42,5 @@
     <parent link="base_link"/>
     <child link="wheel_left_link"/>
-    <origin xyz="0.0 0.08 0.023" rpy="-1.57 0 0"/>
+    <origin xyz="0.0 ${WS/2} 0.023" rpy="-1.57 0 0"/>
     <axis xyz="0 0 1"/>
   </joint>
@@ -48,5 +56,5 @@
       <origin xyz="0 0 0" rpy="0 0 0"/>
       <geometry>
-        <cylinder length="0.018" radius="0.033"/>
+        <cylinder length="0.018" radius="${WR}"/>
       </geometry>
     </collision>
@@ -62,5 +70,5 @@
     <parent link="base_link"/>
     <child link="wheel_right_link"/>
-    <origin xyz="0.0 -0.080 0.023" rpy="-1.57 0 0"/>
+    <origin xyz="0.0 ${-WS/2} 0.023" rpy="-1.57 0 0"/>
     <axis xyz="0 0 1"/>
   </joint>
@@ -76,5 +84,5 @@
       <origin xyz="0 0 0" rpy="0 0 0"/>
       <geometry>
-        <cylinder length="0.018" radius="0.033"/>
+        <cylinder length="0.018" radius="${WR}"/>
       </geometry>
     </collision>
@@ -85,5 +93,5 @@
                iyy="1.1192413e-05" iyz="-1.4400107e-11"
                izz="2.0712558e-05" />
-      </inertial>
+    </inertial>
   </link>
   <joint name="caster_back_joint" type="fixed">
